Commit message: fixed depth subscription for disparity. Random walk semi-working.

File: robot/ros_ws/src/robot_bringup/urdf/robot.urdf.xacro (robot description, xacro)
@@ -43,5 +43,5 @@
   </joint>
   <!-- Left camera -->
-  <link name="left_camera">
+  <link name="left">
     <visual>
       <geometry>
@@ -55,9 +55,9 @@
   <joint name="camera_mount_to_left" type="fixed">
     <parent link="camera_mount"/>
-    <child link="left_camera"/>
+    <child link="left"/>
     <origin xyz="0 -0.05 0" rpy="0 0 0"/>
   </joint>
   <!-- Right camera -->
-  <link name="right_camera">
+  <link name="right">
     <visual>
       <geometry>
@@ -71,5 +71,5 @@
   <joint name="camera_mount_to_right" type="fixed">
     <parent link="camera_mount"/>
-    <child link="right_camera"/>
+    <child link="right"/>
     <origin xyz="0 0.05 0" rpy="0 0 0"/>
   </joint>

Commit message: Put stereo camera TFs in optical frame

File: robot/ros_ws/src/robot_bringup/urdf/robot.urdf.xacro (robot description, xacro)
@@ -56,5 +56,5 @@
     <parent link="camera_mount"/>
     <child link="left"/>
-    <origin xyz="0 -0.05 0" rpy="0 0 0"/>
+    <origin xyz="0 -0.05 0" rpy="-1.5708 0 -1.5708"/>
   </joint>
   <!-- Right camera -->
@@ -72,5 +72,5 @@
     <parent link="camera_mount"/>
     <child link="right"/>
-    <origin xyz="0 0.05 0" rpy="0 0 0"/>
+    <origin xyz="0 0.05 0" rpy="-1.5708 0 -1.5708"/>
   </joint>
   <!-- LiDAR sensor -->
