Commit message: Progress, URDF working. Now need mavlink to work

File: common/ros_packages/robot_descriptions/iris_with_sensors_description/urdf/iris_with_sensors.pegasus.robot.urdf (robot description, URDF)
Before this commit: robot iris_with_sensors.pegasus.robot, 7 links, 4 joints
Links:
- removed link camera_left_OmniverseKitViewportCameraMesh
- removed link camera_right_OmniverseKitViewportCameraMesh
- added link OS1_REV6_128_10hz___512_resolution; collision mesh filename=package://iris_with_sensors_description/meshes/os1_mesh.obj scale=1. 1. 1.; visual mesh filename=package://iris_with_sensors_description/meshes/os1_mesh.obj scale=1. 1. 1.
- added link base_link_ZED_X; collision mesh filename=package://iris_with_sensors_description/meshes/base_link_ZE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 scale=1. 1. 1.; visual mesh filename=package://iris_with_sensors_description/meshes/base_link_ZE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 scale=1. 1. 1.
- added link base_link_body_body_link; collision mesh filename=package://iris_with_sensors_description/meshes/base_link_bo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 scale=1. 1. 1.; visual mesh filename=package://iris_with_sensors_description/meshes/base_link_bo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 scale=1. 1. 1.
- added link rotor0; collision mesh filename=package://iris_with_sensors_description/meshes/rotor0_iris_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 scale=1. 1. 1.; visual mesh filename=package://iris_with_sensors_description/meshes/rotor0_iris_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 scale=1. 1. 1.
- added link rotor1; collision mesh filename=package://iris_with_sensors_description/meshes/rotor1_iris_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 scale=1. 1. 1.; visual mesh filename=package://iris_with_sensors_description/meshes/rotor1_iris_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 scale=1. 1. 1.
- added link rotor2; collision mesh filename=package://iris_with_sensors_description/meshes/rotor2_iris_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 scale=1. 1. 1.; visual mesh filename=package://iris_with_sensors_description/meshes/rotor2_iris_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 scale=1. 1. 1.
- added link rotor3; collision mesh filename=package://iris_with_sensors_description/meshes/rotor3_iris_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 scale=1. 1. 1.; visual mesh filename=package://iris_with_sensors_description/meshes/rotor3_iris_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 scale=1. 1. 1.
- link base_link: geometry 
Joints:
- removed joint joint_base_link-camera_left
- removed joint joint_base_link-camera_right
- removed joint joint_base_link-imu
- removed joint joint_base_link-lidar
- added joint DistanceJoint: type fixed, parent base_link, child base_link_body_body_link, origin xyz=0. 0. 0. rpy=0. 0. 1.5707872
- added joint OS1_REV6_128_10hz___512_resolution_FixedJoint: type fixed, parent base_link_body_body_link, child OS1_REV6_128_10hz___512_resolution, origin xyz=0. 0. 0.0425594 rpy=0. 0. -1.5707872
- added joint base_link_ZED_X_FixedJoint: type fixed, parent base_link_body_body_link, child base_link_ZED_X, origin xyz=0.0000013 -0.1451943 -0.0066019 rpy=0.1745329 0. 0.0000091
- added joint joint0: type continuous, parent base_link_body_body_link, child rotor0, origin xyz=-0.2067341 -0.1375972 0.023  rpy=0. 0. 0., axis 0. 0. 1.
- added joint joint1: type continuous, parent base_link_body_body_link, child rotor1, origin xyz=0.2186935 0.125002 0.023  rpy=0. 0. 0., axis 0. 0. 1.
- added joint joint2: type continuous, parent base_link_body_body_link, child rotor2, origin xyz=0.2032209 -0.138307 0.023  rpy=0. 0. 0., axis 0. 0. 1.
- added joint joint3: type continuous, parent base_link_body_body_link, child rotor3, origin xyz=-0.222 0.1245 0.023  rpy=0. 0. 0., axis 0. 0. 1.
- added joint joint_OS1_REV6_128_10hz___512_resolution-lidar: type fixed, parent OS1_REV6_128_10hz___512_resolution, child lidar, origin xyz=0. 0. 0.03622 rpy=0. 0. -0.
- added joint joint_base_link_ZED_X-camera_left: type fixed, parent base_link_ZED_X, child camera_left, origin xyz=0.05994 -0.00909 0.0134  rpy=1.5707964 0. -3.1415927
- added joint joint_base_link_ZED_X-camera_right: type fixed, parent base_link_ZED_X, child camera_right, origin xyz=-0.05994 -0.00909 0.0134  rpy=1.5707964 0. -3.1415927
- added joint joint_base_link_ZED_X-imu: type fixed, parent base_link_ZED_X, child imu, origin xyz=0.06 0.014058 0.0134  rpy=0. 0. 0.

Commit message: Had to fix camera frame by 180deg rotate about X (following isaac docs)

File: common/ros_packages/robot_descriptions/iris_with_sensors_description/urdf/iris_with_sensors.pegasus.robot.urdf (robot description, URDF)
Before this commit: robot iris_with_sensors.pegasus.robot, 12 links, 11 joints
Joints:
- joint joint_base_link_ZED_X-camera_left: origin xyz=0.05994 -0.00909 0.0134  rpy=1.5707964 0. -3.1415927 -> xyz=0.05994 -0.00909 0.0134  rpy=-1.5707964 0. -3.1415927
- joint joint_base_link_ZED_X-camera_right: origin xyz=-0.05994 -0.00909 0.0134  rpy=1.5707964 0. -3.1415927 -> xyz=-0.05994 -0.00909 0.0134  rpy=-1.5707964 0. -3.1415927

Commit message: Frame updates

File: common/ros_packages/robot_descriptions/iris_with_sensors_description/urdf/iris_with_sensors.pegasus.robot.urdf (robot description, URDF)
Before this commit: robot iris_with_sensors.pegasus.robot, 12 links, 11 joints
Joints:
- joint joint_OS1_REV6_128_10hz___512_resolution-lidar: origin xyz=0. 0. 0.03622 rpy=0. 0. -0. -> xyz=0. 0. 0.03622 rpy=0 1.57 1.57

Commit message: fixing lidar orientation direction in robot description

File: common/ros_packages/robot_descriptions/iris_with_sensors_description/urdf/iris_with_sensors.pegasus.robot.urdf (robot description, URDF)
Before this commit: robot iris_with_sensors.pegasus.robot, 12 links, 11 joints
Joints:
- joint joint_OS1_REV6_128_10hz___512_resolution-lidar: origin xyz=0. 0. 0.03622 rpy=0 1.57 1.57 -> xyz=0. 0. 0.03622 rpy=0 0 1.57

Commit message: fixes to visuals for rviz and robot description based on new default sensor positions

File: common/ros_packages/robot_descriptions/iris_with_sensors_description/urdf/iris_with_sensors.pegasus.robot.urdf (robot description, URDF)
Before this commit: robot iris_with_sensors.pegasus.robot, 12 links, 11 joints
Joints:
- joint OS1_REV6_128_10hz___512_resolution_FixedJoint: origin xyz=0. 0. 0.0425594 rpy=0. 0. -1.5707872 -> xyz=0. 0. 0.15 rpy=0. 0. -1.5707872
- joint base_link_ZED_X_FixedJoint: origin xyz=0.0000013 -0.1451943 -0.0066019 rpy=0.1745329 0. 0.0000091 -> xyz=0.0 -0.2 -0.05 rpy=0. 0. 0.
- joint joint0: type continuous -> fixed
- joint joint1: type continuous -> fixed
- joint joint2: type continuous -> fixed
- joint joint3: type continuous -> fixed

Commit message: Johnliu/pegasus update (#312)
* updated pegasus version, updated docker compose version. Connects robot and px4, but WIP ogn api updates

* Fixed python path in isaac-sim container. Now properly publishes clock and connects to robot for basic flight

* uncommented example script code

* fixing lidar orientation direction in robot description

* updated two_example script as well

* added error message for stale docker compose version

* fixed example script for 2 robots to properly namespace the two different robots

* bump version to 0.16.0 for new Isaac Sim/Pegasus version and on Ubuntu 24

* Update rviz to show lidar

* sync with WIP spawn multirotor node to fix sim-airstack timesync issue

* fixes to visuals for rviz and robot description based on new default sensor positions

* enable proper extension in example script for OnPhysicsStep ogn

* properly does not play scripted environment on start if specified in env file

* Rename ISAAC_SIM_USE_STANDALONE_SCRIPT to ISAAC_SIM_USE_STANDALONE

* Add light to script, add clock display

* Update airstack cli to containerize docker compose itself, so that users don't have to manage different versions

* Bump to docker-compose 5.0.2, also get docker image tag for tagging airstack-cli image

* Fix display forwarding for containerized docker-compose

* Fix env variable propagation in containerized docker-compose

* Small changes

* added environment var to isaac docker compose to properly play sim on start from env file

* temporary fix, airstack with USD file has no wobble; scripted mode still wobbles

* Add ground plane

* update rviz

---------

Co-authored-by: John <John Liu>
Co-authored-by: Andrew Jong <ajong@andrew.cmu.edu>

File: common/ros_packages/robot_descriptions/iris_with_sensors_description/urdf/iris_with_sensors.pegasus.robot.urdf (robot description, URDF)
Before this commit: robot iris_with_sensors.pegasus.robot, 12 links, 11 joints
Joints:
- joint OS1_REV6_128_10hz___512_resolution_FixedJoint: origin xyz=0. 0. 0.0425594 rpy=0. 0. -1.5707872 -> xyz=0. 0. 0.15 rpy=0. 0. -1.5707872
- joint base_link_ZED_X_FixedJoint: origin xyz=0.0000013 -0.1451943 -0.0066019 rpy=0.1745329 0. 0.0000091 -> xyz=0.0 -0.2 -0.05 rpy=0. 0. 0.
- joint joint0: type continuous -> fixed
- joint joint1: type continuous -> fixed
- joint joint2: type continuous -> fixed
- joint joint3: type continuous -> fixed
- joint joint_OS1_REV6_128_10hz___512_resolution-lidar: origin xyz=0. 0. 0.03622 rpy=0 1.57 1.57 -> xyz=0. 0. 0.03622 rpy=0 0 1.57

Commit message: Fully automated standalone mode. Added lidar minRange parameter in standalone generation. Kills/restarts PX4 when timeline stops.

File: common/ros_packages/robot_descriptions/iris_with_sensors_description/urdf/iris_with_sensors.pegasus.robot.urdf (robot description, URDF)
Before this commit: robot iris_with_sensors.pegasus.robot, 12 links, 11 joints
Joints:
- joint OS1_REV6_128_10hz___512_resolution_FixedJoint: origin xyz=0. 0. 0.15 rpy=0. 0. -1.5707872 -> xyz=0. 0. 0.025 rpy=0. 0. -1.5707872
