Commit message: Robot builds and launches again

File: ros_ws/src/robot_descriptions/iris/urdf/iris_with_sensors.pegasus.robot.urdf (robot description, URDF)
Before this commit: robot iris_with_sensors.pegasus.robot, 12 links, 11 joints
Links:
- link OS1_REV6_128_10hz___512_resolution: geometry collision mesh filename=package://robot_descriptions/iris/meshes/os1_mesh.obj scale=1. 1. 1.; visual mesh filename=package://robot_descriptions/iris/meshes/os1_mesh.obj scale=1. 1. 1.
- link base_link_ZED_X: geometry collision mesh filename=package://robot_descriptions/iris/meshes/base_link_ZED_X_ba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 scale=1. 1. 1.; visual mesh filename=package://robot_descriptions/iris/meshes/base_link_ZED_X_ba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 scale=1. 1. 1.
- link base_link_body_body_link: geometry collision mesh filename=package://robot_descriptions/iris/meshes/base_link_body_bod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 scale=1. 1. 1.; visual mesh filename=package://robot_descriptions/iris/meshes/base_link_body_bod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 scale=1. 1. 1.
- link rotor0: geometry collision mesh filename=package://robot_descriptions/iris/meshes/rotor0_iris_prop_c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 scale=1. 1. 1.; visual mesh filename=package://robot_descriptions/iris/meshes/rotor0_iris_prop_c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 scale=1. 1. 1.
- link rotor1: geometry collision mesh filename=package://robot_descriptions/iris/meshes/rotor1_iris_prop_c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 scale=1. 1. 1.; visual mesh filename=package://robot_descriptions/iris/meshes/rotor1_iris_prop_c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 scale=1. 1. 1.
- link rotor2: geometry collision mesh filename=package://robot_descriptions/iris/meshes/rotor2_iris_prop_c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 scale=1. 1. 1.; visual mesh filename=package://robot_descriptions/iris/meshes/rotor2_iris_prop_c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 scale=1. 1. 1.
- link rotor3: geometry collision mesh filename=package://robot_descriptions/iris/meshes/rotor3_iris_prop_c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 scale=1. 1. 1.; visual mesh filename=package://robot_descriptions/iris/meshes/rotor3_iris_prop_c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 scale=1. 1. 1.
