Commit message: removed deprecated ouster lidar. Completely integrated new rtx lidar

File: common/ros_packages/robot_descriptions/iris/urdf/iris_with_sensors.pegasus.robot.urdf (robot description, URDF)
Before this commit: robot iris_with_sensors.pegasus.robot, 12 links, 11 joints
Links:
- removed link OS1_REV6_128_10hz___512_resolution
- added link lidar_mount; collision mesh filename=package://robot_descriptions/iris/meshes/os1_mesh.obj scale=1. 1. 1.; visual mesh filename=package://robot_descriptions/iris/meshes/os1_mesh.obj scale=1. 1. 1.
Joints:
- removed joint OS1_REV6_128_10hz___512_resolution_FixedJoint
- removed joint joint_OS1_REV6_128_10hz___512_resolution-lidar
- added joint base_link_body_to_lidar_mount: type fixed, parent base_link_body_body_link, child lidar_mount, origin xyz=0. 0. 0.025 rpy=0. 0. -1.5707872
- added joint lidar_mount_to_lidar: type fixed, parent lidar_mount, child lidar, origin xyz=0. 0. 0.05 rpy=0 0 1.57

Commit message: Update PegasusSim lidar to new rtx lidar and optional min_sensor_range parameter to vdb model to avoid self-detection.

File: common/ros_packages/robot_descriptions/iris/urdf/iris_with_sensors.pegasus.robot.urdf (robot description, URDF)
Before this commit: robot iris_with_sensors.pegasus.robot, 12 links, 11 joints
Joints:
- joint joint_OS1_REV6_128_10hz___512_resolution-lidar: origin xyz=0. 0. 0.03622 rpy=0 0 1.57 -> xyz=0. 0. 0.05 rpy=0 0 1.57

Commit message: renaming frame id back to ouster

File: common/ros_packages/robot_descriptions/iris/urdf/iris_with_sensors.pegasus.robot.urdf (robot description, URDF)
Before this commit: robot iris_with_sensors.pegasus.robot, 12 links, 11 joints
Links:
- removed link lidar
- added link ouster
Joints:
- removed joint lidar_mount_to_lidar
- added joint lidar_mount_to_ouster: type fixed, parent lidar_mount, child ouster, origin xyz=0. 0. 0.05 rpy=0 0 1.57
