Commit message: Johnliu/rtx lidar update (#351)
* Update PegasusSim lidar to new rtx lidar and optional min_sensor_range parameter to vdb model to avoid self-detection.

* removed deprecated ouster lidar. Completely integrated new rtx lidar

* renaming frame id back to ouster

* Added node to filter near and invalid lidar points

* reconciled topic names for lidar point cloud

* fixed example scripts to use rtx lidar api

* fixed tmux closing and rclpy path issue

* uses add_rtx in multi px4 script

* bumping version index

* docs added

* unit testing and documentation updates

* cleaning code from copilot suggestions

* docs(tests): fix pytest marker example for running liveliness and sensors

Agent-Logs-Url: https://github.com/castacks/AirStack/sessions/7ce7609a-a7f3-414d-9d42-0c9999d0459f

Co-authored-by: andrewjong <8121216+andrewjong@users.noreply.github.com>

* docs(tests): fix marker semantics in test_sensors module docstring

Agent-Logs-Url: https://github.com/castacks/AirStack/sessions/bdf00f6f-1d9f-4597-bf57-b96f99421646

Co-authored-by: andrewjong <8121216+andrewjong@users.noreply.github.com>

* addressing github copilot concerns

* docs(bridge): remove stale camera topics comment

Agent-Logs-Url: https://github.com/castacks/AirStack/sessions/2d5718ac-20e3-4f10-a12e-05d601cf000c

Co-authored-by: JohnYanxinLiu <63010779+JohnYanxinLiu@users.noreply.github.com>

* addressing copilot concerns

* removing debug print statement from reading point cloud

Co-authored-by: Copilot Autofix powered by AI <175728472+Copilot@users.noreply.github.com>

* fix(isaac-sim): align drone1 lidar prim path with spawned prim

Agent-Logs-Url: https://github.com/castacks/AirStack/sessions/fbad2b9c-1761-45b1-b464-3e874511255c

Co-authored-by: JohnYanxinLiu <63010779+JohnYanxinLiu@users.noreply.github.com>

* more succint comment in sim bashrc

* resolving discrepant comments in ros bridge yaml

* removed bug allocated new copy of point cloud array

* logs lidaar test with boolean instead of hz

* and --> or for marks

---------

Co-authored-by: copilot-swe-agent[bot] <198982749+Copilot@users.noreply.github.com>
Co-authored-by: andrewjong <8121216+andrewjong@users.noreply.github.com>
Co-authored-by: Copilot Autofix powered by AI <175728472+Copilot@users.noreply.github.com>
Co-authored-by: Andrew Jong <ajong@andrew.cmu.edu>

File: common/ros_packages/robot_descriptions/iris/urdf/iris_with_sensors.pegasus.robot.urdf (robot description, URDF)
Before this commit: robot iris_with_sensors.pegasus.robot, 12 links, 11 joints
Links:
- removed link OS1_REV6_128_10hz___512_resolution
- removed link lidar
- added link lidar_mount; collision mesh filename=package://robot_descriptions/iris/meshes/os1_mesh.obj scale=1. 1. 1.; visual mesh filename=package://robot_descriptions/iris/meshes/os1_mesh.obj scale=1. 1. 1.
- added link ouster
Joints:
- removed joint OS1_REV6_128_10hz___512_resolution_FixedJoint
- removed joint joint_OS1_REV6_128_10hz___512_resolution-lidar
- added joint base_link_body_to_lidar_mount: type fixed, parent base_link_body_body_link, child lidar_mount, origin xyz=0. 0. 0.025 rpy=0. 0. -1.5707872
- added joint lidar_mount_to_ouster: type fixed, parent lidar_mount, child ouster, origin xyz=0. 0. 0.05 rpy=0 0 1.57
