Commit message: feat: qualify RRM visual evidence and reconcile Isaac camera frames

File: common/ros_packages/robot_descriptions/iris/urdf/iris_with_sensors.pegasus.robot.urdf (robot description, URDF)
Before this commit: robot iris_with_sensors.pegasus.robot, 12 links, 11 joints
Joints:
- joint joint_base_link_ZED_X-camera_left: origin xyz=0.05994 -0.00909 0.0134  rpy=-1.5707964 0. -3.1415927 -> xyz=0.06 -0.015 0.015 rpy=-1.5707964 0. -3.1415927
- joint joint_base_link_ZED_X-camera_right: origin xyz=-0.05994 -0.00909 0.0134  rpy=-1.5707964 0. -3.1415927 -> xyz=-0.06 -0.015 0.015 rpy=-1.5707964 0. -3.1415927
