Commit message: livox config

File: robot/ros_ws/src/autonomy/4_global/b_planners/integrated_planner/config/model_ai_extrinsics.urdf (robot description, URDF)
Before this commit: robot voxl_extrinsics, 12 links, 11 joints
Links:
- added link livox
Joints:
- added joint imu_to_livox: type fixed, parent imu_apps, child livox, origin xyz=0.01315 -0.01100 0.01047 rpy=-0.5148722 0 -1.5707963
